File: IO.kicad_pcb (KiCad board)
At the start: 2 copper layers, 95 x 72 mm, 31 parts, among them CN1 DC5V1, CN2 Nu UART2 Ctrl, CN3 Alt TEST SW, U1 MAX232

Commit message: some change
Connections:
- CN3 pad 1: Net-(CN3-Pad1) -> GND
- CN3 pad 2: GND -> Net-(CN3-Pad2)
- Nano1 pad 12: Net-(CN3-Pad1) -> Net-(CN3-Pad2)
- OP_U1 pad 15: Net-(CN3-Pad1) -> Net-(CN3-Pad2)
- TEST_SW1 pad 1: Net-(CN3-Pad1) -> Net-(CN3-Pad2)
- TEST_SW1 pad 2: Net-(CN3-Pad1) -> Net-(CN3-Pad2)
Routing:
- net Net-(CN3-Pad1): track 84.3 -> 0.00 mm
- net Net-(CN3-Pad2): track 0.00 -> 81.8 mm

Commit message: r3 beta
Routing:
- net Net-(CN2-Pad3): track 107.5 -> 108.6 mm
- net Net-(OP_CN4-Pad1): track 15.7 -> 16.5 mm
Changed lines of the file:
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@@
     (thickness 1.6)
     (drawings 27)
-    (tracks 481)
+    (tracks 484)
     (zones 0)
     (modules 31)
@@
   )
   (page A4)
+  (title_block
+    (title REVIO)
+    (date 2021-03-25)
+    (rev r3)
+    (company NTSK-Lab)
+  )
   (layers
     (0 F.Cu signal)
@@
   (via (at 145.415 57.15) (size 0.8) (drill 0.4) (layers F.Cu B.Cu) (net 8))
   (via (at 145.415 59.69) (size 0.8) (drill 0.4) (layers F.Cu B.Cu) (net 8))
-  (segment (start 145.415 59.69) (end 145.415 90.805) (width 0.25) (layer F.Cu) (net 8))
-  (segment (start 147.868 93.258) (end 149.352 93.258) (width 0.25) (layer F.Cu) (net 8))
-  (segment (start 145.415 90.805) (end 147.868 93.258) (width 0.25) (layer F.Cu) (net 8))
   (segment (start 133.985 46.355) (end 133.985 56.515) (width 0.25) (layer F.Cu) (net 8))
   (segment (start 133.985 56.515) (end 134.62 57.15) (width 0.25) (layer F.Cu) (net 8))
@@
   (segment (start 125.175 57.705) (end 125.175 53.975) (width 0.25) (layer F.Cu) (net 8))
   (segment (start 122.645 79.375) (end 121.285 79.375) (width 0.25) (layer F.Cu) (net 8))
+  (segment (start 145.415 89.535) (end 145.415 59.69) (width 0.25) (layer F.Cu) (net 8))
+  (segment (start 145.963 93.258) (end 145.415 92.71) (width 0.25) (layer F.Cu) (net 8))
+  (segment (start 145.415 92.71) (end 145.415 89.535) (width 0.25) (layer F.Cu) (net 8))
+  (segment (start 149.352 93.258) (end 145.963 93.258) (width 0.25) (layer F.Cu) (net 8))
   (segment (start 146.685 90.17) (end 147.32 90.805) (width 0.25) (layer F.Cu) (net 9))
   (segment (start 146.685 59.055) (end 146.685 90.17) (width 0.25) (layer F.Cu) (net 9))
@@
   (segment (start 153.67 60.325) (end 153.67 71.19) (width 0.25) (layer B.Cu) (net 24))
   (segment (start 151.765 59.73) (end 153.075 59.73) (width 0.25) (layer B.Cu) (net 24))
+  (segment (start 147.972 73.008) (end 149.352 73.008) (width 0.25) (layer F.Cu) (net 25))
+  (segment (start 147.955 73.025) (end 147.972 73.008) (width 0.25) (layer F.Cu) (net 25))
+  (segment (start 147.32 62.865) (end 147.32 72.39) (width 0.25) (layer F.Cu) (net 25))
+  (segment (start 147.32 72.39) (end 147.955 73.025) (width 0.25) (layer F.Cu) (net 25))
+  (segment (start 147.955 62.23) (end 147.32 62.865) (width 0.25) (layer F.Cu) (net 25))
   (segment (start 151.765 62.23) (end 147.955 62.23) (width 0.25) (layer F.Cu) (net 25))
-  (segment (start 147.955 62.23) (end 147.32 62.865) (width 0.25) (layer F.Cu) (net 25))
-  (segment (start 147.32 70.976) (end 149.352 73.008) (width 0.25) (layer F.Cu) (net 25))
-  (segment (start 147.32 62.865) (end 147.32 70.976) (width 0.25) (layer F.Cu) (net 25))
   (segment (start 152.988 90.758) (end 151.852 90.758) (width 0.25) (layer F.Cu) (net 26))
   (segment (start 153.67 98.425) (end 153.67 91.44) (width 0.25) (layer F.Cu) (net 26))

Commit message: move silk
Parts:
- Nano1: value Arduino_Nano_v3.x -> Arduino_Nano
Other:
- board text added: "+"
- board text added: "1"

Commit message: kicad 6.x
Other:
- net class Default removed
